File: Schaltungen/LED-Platine/2018_01_31_neu/circuit/gluecksrad.brd (EAGLE design)
At the start: 100 x 40 mm, 17 parts, among them IC1 LOGIK_SHIFT8, IC2 ULN2003AD

Commit message: updated LED-Platine (resistor for red is 150R not 120R)
Parts:
- R1, R4: value 120 -> 150
Changed lines of the file:
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@@
 <attribute name="VALUE" x="45.936" y="19.685" size="1.27" layer="28" ratio="10" rot="MR180"/>
 </element>
-<element name="R1" library="robo_ag" package="R_THT_4" value="120" x="33.02" y="20.32" smashed="yes">
+<element name="R1" library="robo_ag" package="R_THT_4" value="150" x="33.02" y="20.32" smashed="yes">
 <attribute name="VALUE" x="33.02" y="17.145" size="1.27" layer="27" ratio="10" align="bottom-center"/>
 </element>
@@
 <attribute name="VALUE" x="33.02" y="22.225" size="1.27" layer="27" ratio="10" align="bottom-center"/>
 </element>
-<element name="R4" library="robo_ag" package="R_THT_4" value="120" x="67.31" y="25.4" smashed="yes">
+<element name="R4" library="robo_ag" package="R_THT_4" value="150" x="67.31" y="25.4" smashed="yes">
 <attribute name="VALUE" x="67.31" y="22.225" size="1.27" layer="27" ratio="10" align="bottom-center"/>
 </element>
