File: Schaltungen/LED-Platine/2018_01_31_neu/circuit/gluecksrad.sch (EAGLE design)
At the start: 17 parts, among them IC1 LOGIK_SHIFT8, IC2 ULN2003AD

Commit message: updated LED-Platine (resistor for red is 150R not 120R)
Parts:
- R1, R4: value 120 -> 150
Changed lines of the file:
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@@
 <part name="P+3" library="supply1" deviceset="+5V" device=""/>
 <part name="P+4" library="supply1" deviceset="+5V" device=""/>
-<part name="R1" library="robo_ag" deviceset="RESISTOR" device="-10MM" value="120"/>
+<part name="R1" library="robo_ag" deviceset="RESISTOR" device="-10MM" value="150"/>
 <part name="R2" library="robo_ag" deviceset="RESISTOR" device="-10MM" value="100"/>
 <part name="R3" library="robo_ag" deviceset="RESISTOR" device="-10MM" value="100"/>
 <part name="P+5" library="supply1" deviceset="+5V" device=""/>
-<part name="R4" library="robo_ag" deviceset="RESISTOR" device="-10MM" value="120"/>
+<part name="R4" library="robo_ag" deviceset="RESISTOR" device="-10MM" value="150"/>
 <part name="R5" library="robo_ag" deviceset="RESISTOR" device="-10MM" value="100"/>
 <part name="R6" library="robo_ag" deviceset="RESISTOR" device="-10MM" value="100"/>
